Commit message: 5

File: real_car/urdf/real_car.urdf (robot description, URDF)
Before this commit: robot real_car, 44 links, 43 joints
Links:
- link ls1: mass 2.6548E-05 -> 0.001
- link ls2: mass 2.65475633543081E-05 -> 0.001
- link ls3: mass 2.65475633543081E-05 -> 0.001
- link ls4: mass 2.65475633543081E-05 -> 0.001
- link rs1: mass 2.65475633543081E-05 -> 0.001
- link rs2: mass 2.65475633543081E-05 -> 0.001
- link rs3: mass 2.65475633543081E-05 -> 0.001
- link rs4: mass 2.65475633543081E-05 -> 0.001
